Commit message: added lhm differential controller

File: robbie_description/urdf/lhm/lhm.transmission.xacro (robot description, xacro)
@@ -4,7 +4,4 @@
 		<transmission name="lhm_${side}_transmission">
 			<type>transmission_interface/SimpleTransmission</type>
-			<!-- FOR HYDRO -->  <!--
-			<joint name="lhm_wheel_${side}_joint"/>
-			-->
 			<!-- FOR INDIGO -->
 			<joint name="lhm_wheel_${side}_joint">
