Commit message: update to robot description and sensors

File: robbie_description/urdf/lhm/lhm.xacro (robot description, xacro)
@@ -53,5 +53,5 @@
 		<!-- lhm link -->
 		<link name="lhm_link">
-			<collision>
+			<collision name = "lhm_link">
 				<origin rpy="0 0 0" xyz="0 0 0"/>
 				<geometry>
@@ -71,7 +71,9 @@
 			</inertial>
 		</link>
+<!--
 		<gazebo reference="lhm_link">
 			<material>Gazebo/White</material>
 		</gazebo>
+ -->
 		<joint name="lhm_torso_joint" type="prismatic">
 			<origin rpy="0 0 0" xyz="-0.03 0 -0.05"/>
@@ -80,5 +82,5 @@
 			<axis xyz="0 0 1"/>
 			<dynamics damping="1"/>
-			<limit effort="300" lower="-.2" upper="0" velocity="0.1"/>
+			<limit effort="300" lower="-.4" upper="0" velocity="0.1"/>
 		</joint>
 	<!-- declare two shank wheels -->

File: robbie_description/urdf/sensors/sensors.xacro (robot description, xacro)
@@ -30,5 +30,5 @@
   </joint>
   <!-- Hokuyo Laser -->
-  <link name="hokuyo_link">
+<!--   <link name="hokuyo_link">
     <collision>
       <origin xyz="0 0 0" rpy="0 0 0"/>
@@ -49,11 +49,92 @@
     </inertial>
   </link>
-  <joint name="hokuyo_joint" type="fixed">
+ -->
+<!--   <link name="shank_proximity_link">
+    <visual>
+      <origin xyz="0 0 0" rpy="0 0 0"/>
+      <geometry>
+        <mesh filename="package://robbie_description/meshes/kinect.dae" scale="0.8 0.8 0.8"/>
+      </geometry>
+    </visual>
+    <inertial>
+      <mass value="1e-5" />
+      <origin xyz="0 0 0" rpy="0 0 0"/>
+      <inertia ixx="1e-6" ixy="0" ixz="0" iyy="1e-6" iyz="0" izz="1e-6" />
+    </inertial>
+  </link>
+ -->
+<!--   <joint name="hokuyo_joint" type="fixed">
     <axis xyz="0 1 0" />
-    <origin xyz="0 0 0.4" rpy="0 -1.22173048 0"/>
+    <origin xyz="0 0 0.4" rpy="1.57 -1.22173048 0"/>
     <parent link="shank_link"/>
     <child link="hokuyo_link"/>
+    <limit effort="300" lower="0" upper="1.5" velocity="0.01"/>
   </joint>
-  <!--link name="kinect_link">
+ -->
+<!--   <joint name="shank_kinect_joint" type="fixed">
+    <axis xyz="0 1 0" />
+    <origin xyz="0.08 0 0.17350" rpy="0 0 0"/>
+    <parent link="shank_link"/>
+    <child link="shank_proximity_link"/>
+    <limit effort="300" lower="0" upper="1.5" velocity="0.01"/>
+  </joint>
+ -->
+<!--   <joint name="shank_kinect_optical_joint" type="fixed">
+    <origin xyz="0 0 0" rpy="-1.57 0 -1.57"/>
+    <parent link="shank_proximity_link"/>
+    <child link="shank_kinect_optical_frame"/>
+  </joint>
+  <link name="shank_kinect_optical_frame"/>
+ -->
+<!--   <joint name="shank_hokuyo_joint" type="fixed">
+    <axis xyz="0 0 1" />
+    <origin xyz="0.1 0 0.17350" rpy="-1.57 0 0"/>
+    <parent link="shank_link"/>
+    <child link="shank_proximity_link"/>
+    <limit effort="300" lower="0" upper="1.5" velocity="0.01"/>
+  </joint>
+ -->
+<!--       <geometry>
+    <box size="0.1 0.1 0.1"/>
+      </geometry>
+ -->
+<!--   <link name="stab_contact_link">
+      <collision name="stab_contact">
+        <origin rpy="0 0 0" xyz="0 0 0"/>
+        <geometry>
+         <mesh filename="package://robbie_description/meshes/stabiliserWheel_collision.stl"/>
+        </geometry>
+      </collision>
+    <visual>
+      <origin xyz="0 0 0" rpy="0 0 0" />
+      <geometry>
+        <sphere radius="0.1"/>
+        <mesh filename="package://robbie_description/meshes/stabiliserWheel.stl" scale="1 1 1"/>
+        <cylinder radius="0.01" length="0.05"/>
+      </geometry>
+    </visual>
+    <inertial>
+      <mass value="0" />
+      <origin xyz="0 0 0" rpy="0 0 0"/>
+      <inertia ixx="0" ixy="0" ixz="0" iyy="0" iyz="0" izz="0" />
+    </inertial>
+  </link>
+ -->
+<!--   <joint name="stab_sensor_joint" type="fixed">
+    <axis xyz="0 0 0" />
+    <origin xyz="0.4 0 0" rpy="0 0 0"/>
+    <parent link="stab_wheel"/>
+    <child link="stab_contact_link"/>
+  </joint>
+ -->
+<!--
+  <joint name="stabWheel_sensor_joint" type="fixed">
+    <origin rpy="0 0 0" xyz="-0.1 0 .2"/>
+    <parent link="stab_link"/>
+    <child link="stab_contact_link"/>
+    <axis xyz="0 1 0"/>
+  </joint>
+ -->
+<!--   <link name="kinect_link">
     <collision>
       <origin xyz="0 0 0" rpy="0 0 0"/>
@@ -73,4 +154,5 @@
       <inertia ixx="1e-6" ixy="0" ixz="0" iyy="1e-6" iyz="0" izz="1e-6" />
     </inertial>
-  </link-->
+  </link>
+ -->
 </robot>

File: robbie_description/urdf/shank/shank.xacro (robot description, xacro)
@@ -73,7 +73,8 @@
 			</inertial>
 		</link>
-		<gazebo reference="${name}_link">
+<!-- 		<gazebo reference="${name}_link">
 			<material>Gazebo/White</material>
 		</gazebo>
+ -->
 		<!-- footprint-shank joint -->
 		<joint name="${name}_footprint_joint" type="fixed">

File: robbie_description/urdf/stabiliser/stabiliser.xacro (robot description, xacro)
@@ -64,5 +64,5 @@
 			<mu1>0.0</mu1>
 			<mu2>0.0</mu2>
-		</gazebo>
+ 		</gazebo>
 		<joint name="stab_joint" type="revolute">
 			<origin rpy="0 0.698131701 0" xyz="0 0 .24"/>

Commit message: added contact sensors

File: robbie_description/urdf/lhm/lhm.xacro (robot description, xacro)
@@ -15,5 +15,5 @@
   <xacro:macro name="lhm_wheel" params="side reflect" parent="lhm_link">
 		<link name="lhm_wheel_${side}_link">
-			<collision>
+			<collision name="lhm_wheel_${side}_link_collision">
 				<origin rpy="0 0 0" xyz="0 0 0"/>
 				<geometry>
@@ -37,7 +37,8 @@
 		</link>
 		<!--gazebo defns-->
-		<gazebo reference="lhm_wheel_${side}_link">
+<!-- 		<gazebo reference="lhm_wheel_${side}_link">
 			<material>Gazebo/Black</material>
 		</gazebo>
+ -->
 		<!-- define shank-wheel joint -->
 		<joint name="lhm_wheel_${side}_joint" type="continuous">

File: robbie_description/urdf/shank/shank.xacro (robot description, xacro)
@@ -14,5 +14,5 @@
   <xacro:macro name="shank_wheel" params="side reflect" parent="shank_link">
 		<link name="wheel_${side}_link">
-			<collision>
+			<collision name="wheel_${side}_link_collision">
 				<origin rpy="0 0 0" xyz="0 0 0"/>
 				<geometry>
@@ -36,7 +36,19 @@
 		</link>
 		<!--gazebo defns-->
-		<gazebo reference="wheel_${side}_link">
+<!-- 		<gazebo reference="wheel_${side}_link">
 			<material>Gazebo/Black</material>
+			<sensor type="contact" name="wheel_${side}_contact">
+				<contact>
+					<collision>wheel_${side}_collision_collision</collision>
+				</contact>
+				<plugin name="gazebo_ros_bumper_controller" filename="libgazebo_ros_bumper.so">
+					<bumperTopicName>robbie/wheel_${side}/contact</bumperTopicName>
+					<frameName>wheel_${side}_link</frameName>
+					<alwaysOn>true</alwaysOn>
+					<updateRate>5</updateRate>
+				</plugin>
+			</sensor>
 		</gazebo>
+ -->
 		<!-- define shank-wheel joint -->
 		<joint name="wheel_${side}_joint" type="continuous">

File: robbie_description/urdf/stabiliser/stabiliser.xacro (robot description, xacro)
@@ -39,5 +39,5 @@
 		</gazebo>
 		<link name="stab_wheel">
-			<collision>
+			<collision name="stab_wheel_collision">
 				<origin rpy="0 0 0" xyz="0 0 0"/>
 				<geometry>
@@ -60,9 +60,10 @@
 			</inertial>
 		</link>
-		<gazebo reference="stab_wheel">
+<!-- 		<gazebo reference="stab_wheel">
 			<material>Gazebo/Black</material>
 			<mu1>0.0</mu1>
 			<mu2>0.0</mu2>
  		</gazebo>
+ -->
 		<joint name="stab_joint" type="revolute">
 			<origin rpy="0 0.698131701 0" xyz="0 0 .24"/>
